File: overallPCB.sch (EAGLE design)
At the start: 41 parts, among them IC4 CP2104, IC7 DS3231/SO, Q7 mmbt2222, Q8 mmbt2222, Q9 DMG3415U, SW3 KMR2, U5 MCP73831T-2ACI/OT, U6 AP2112-3.3, U7 TB6621FNG, X7 ESP32_WROOM32_SKINNY, X8 20329, X9 JSTPH

Commit message: Add files via upload
Parts:
- removed D6: RED, microbuilder:LED0805_NOOUTLINE
- removed R29: 1K, microbuilder:RESISTOR_0603_NOOUT
- added J3: (no value), SparkFun-Connectors:CONN_10"
Connections:
- removed net !RTC_RST: IC7./RST
- removed net 32KHZ: IC7.32KHZ
- removed net MISO: X7.IO19
- removed net N$27: D6.A, R29.2
- removed net SQW: IC7.SQW/INT
- new net GPIO19: J3.3, X7.IO19
- new net N$1: J3.1
- new net N$2: J3.2
- net A0_DAC2: now also J3.6
- net A4_IO36: now also J3.5
- net EN: now also J3.10
- net GND: no longer D6.C
- net IO13_A12: now also J3.4; no longer R29.1
- net RESET: now also J3.9
- net VBAT: now also J3.7
- net VBUS: now also J3.8
Other:
- note removed: "LED"
- moved on the sheet: R22, R23

Commit message: update overallPCB
Parts:
- removed C23: 10uF, SparkFun-Capacitors:10UF-0805-10V-10%
- removed R30: 10k, SparkFun-Resistors:10KOHM-HORIZ-1/4W-5%
- removed U7: TB6621FNG, SparkFun:TB6621FNG
- added C1: 10µF, microbuilder:CAP_CERAMIC0805-NOOUTLINE
- added R2: 10K, microbuilder:RESISTOR0805_NOOUTLINE
- added U2: TB6612 SSOP, microbuilder:TB6612FNGSSOP
Connections:
- removed net A2_I34: X7.I34/A1_6
- removed net A3_I39: X7.IO39/SEN_VN/A1_3
- removed net GPIO2: X7.IO2/A2_2
- removed net N$1: J3.1
- removed net N$2: J3.2
- removed net N$28: R30.1
- removed net N$34: R35.1
- removed net N$35: R36.1
- removed net OLED_TX: J1.8
- new net STBY: R2.1, U2.STBY
- net 3.3V: now also C1.1, J3.1, R2.2, R35.1, R36.1, U2.VCC; no longer C23.1, R30.2
- net AIN1: now also U2.AIN1; no longer U7.AIN2
- net AIN2: now also U2.AIN2; no longer U7.AIN1
- net FINGERPRINT_TX: now also J1.8
- net GND: now also C1.2, J3.2, U2.GND@1, U2.PGND1@1, U2.PGND1@2, U2.PGND2@1, U2.PGND2@2; no longer C23.2, U7.GND, U7.PGND1@3, U7.PGND1@4, U7.PGND2@10, U7.PGND2@9
- net MA1: now also U2.AOUT1@1, U2.AOUT1@2
- net MA2: now also U2.AOUT2@1, U2.AOUT2@2; no longer U7.A02@5, U7.A02@6
- net PWMA: now also U2.PWMA; no longer U7.PWMA
- net VM+: now also U2.VM@1, U2.VM@2, U2.VM@3; no longer U7.VM2, U7.VM3

Commit message: Add files via upload
Parts:
- removed B4: CR1220, microbuilder:BATTERYCR1220_SMT
- removed C28: 1uF, microbuilder:CAP_CERAMIC0805-NOOUTLINE
- removed IC7: DS3231/SO, adafruit:DS3231/SO
- removed R35, R36: 10K, microbuilder:RESISTOR0805_NOOUTLINE
- added B1: CR1220, microbuilder:BATTERYCR1220_SMT
- added C2: 1uF, microbuilder:CAP_CERAMIC0805-NOOUTLINE
- added IC1: DS3231/SO, adafruit:DS3231/SO
- added R1, R3: 10K, microbuilder:RESISTOR0805_NOOUTLINE
Connections:
- net 3.3V: now also C2.2, IC1.VCC, R1.1, R3.1; no longer C28.2, IC7.VCC, R35.1, R36.1
- net GND: now also B1.-, C2.1, IC1.GND; no longer B4.-, C28.1, IC7.GND
- net SCL: now also IC1.SCL, R1.2; no longer IC7.SCL, R35.2
- net SDA: now also IC1.SDA, R3.2; no longer IC7.SDA, R36.2
- net VBAT: now also B1.+, IC1.VBAT; no longer B4.+, IC7.VBAT
Other:
- note added: "MOTOR CONTROLER"
- note added: "RTC"
- moved on the sheet: IC4G$2, Q7, Q8, R21G$2, R21G$4
