File: overallPCB.sch (EAGLE design)
At the start: 40 parts, among them IC1 DS3231/SO, IC4 CP2104, Q7 mmbt2222, Q8 mmbt2222, Q9 DMG3415U, SW3 KMR2, U2 TB6612 SSOP, U5 MCP73831T-2ACI/OT, U6 AP2112-3.3, X7 ESP32_WROOM32_SKINNY, X8 20329, X9 JSTPH

Commit message: Add files via upload
Connections:
- net 3.3V: now also J3.3; no longer J3.1
- net A0_DAC2: now also J3.1; no longer J3.6
- net CONTROL_BUTTON: now also J1.7; no longer J1.2
- net EN: now also J3.9; no longer J3.10
- net FINGERPRINT_RX: now also J1.5; no longer J1.7
- net FINGERPRINT_TX: now also J1.6; no longer J1.8
- net GND: now also J3.4; no longer J3.2
- net GPIO19: now also J3.10; no longer J3.3
- net IO13_A12: now also J3.8; no longer J3.4
- net MOTOR_C1: now also J1.1; no longer J1.9
- net MOTOR_C2: now also J1.4; no longer J1.10
- net OLED_CS: now also J1.9; no longer J1.6
- net OLED_DC: now also J1.3; no longer J1.5
- net OLED_MOSI: now also J1.10; no longer J1.4
- net OLED_SCK: now also J1.8; no longer J1.3
- net RESET: now also J3.2; no longer J3.9
- net SCANNER_BUTTON: now also J1.2; no longer J1.1
- net VBUS: now also J3.6; no longer J3.8

Commit message: Add files via upload
Parts:
- removed J2: (no value), SparkFun-Connectors:CONN_03POGO_PIN_HOLES_ONLY
- removed X8: 20329, microbuilder:USB_MICRO_20329_V2
- added H1, H2: STAND-OFF, SparkFun-Hardware:STAND-OFF
- added J4: (no value), SparkFun-Connectors:CONN_03
- added J5: (no value), SparkFun-Connectors:USB_MICRO-B_FEMALE-SMT
Connections:
- removed net N$21: IC4G$1.D+, X8.D+
- removed net N$22: IC4G$1.D-, X8.D-
- new net N$1: IC4G$1.D+, J5.D+
- new net N$2: IC4G$1.D-, J5.D-
- net EN: now also J3.8; no longer J3.9
- net GND: now also J5.GND; no longer X8.GND
- net IO13_A12: now also J3.7; no longer J3.8
- net MA1: now also J4.2; no longer J2.2
- net MA2: now also J4.3; no longer J2.1
- net VBAT: now also J3.9; no longer J3.7
- net VBUS: now also J5.VBUS; no longer X8.VBUS
- net VM+: now also J4.1; no longer J2.3
