File: overallPCB.sch (EAGLE design)
At the start: 45 parts, among them IC1 DS3231/SO, IC4 CP2104, Q7 mmbt2222, Q8 mmbt2222, Q9 DMG3415U, SW3 KMR2, U2 TB6612 SSOP, U5 MCP73831T-2ACI/OT, U6 AP2112-3.3, X7 ESP32_WROOM32_SKINNY, X8 20329, X9 JSTPH

Commit message: Add files via upload
Parts:
- removed H3, H4: STAND-OFF, SparkFun-Hardware:STAND-OFF
- removed X8: 20329, microbuilder:USB_MICRO_20329_V2
- added X1: Micro USB, SparkFun:USBSMD
Connections:
- net 3.3V: now also J5.4; no longer J5.6
- net EN: now also J5.5; no longer J5.4
- net GND: now also J5.3, X1.GND; no longer J5.5, X8.GND
- net N$21: now also X1.D+; no longer X8.D+
- net N$22: now also X1.D-; no longer X8.D-
- net RESET: now also J5.1; no longer J5.3
- net VBAT: now also J5.6; no longer J5.1
- net VBUS: now also X1.VBUS; no longer X8.VBUS
Other:
- note added: "miniUSB"
Changed lines of the file:
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@@
 <part name="FRAME5" library="frames" library_urn="urn:adsk.eagle:library:229" deviceset="FRAME_C_L" device=""/>
 <part name="IC4" library="microbuilder" deviceset="CP2104" device="" value="CP2104"/>
-<part name="X8" library="microbuilder" deviceset="USB" device="_MICRO_20329_V2" value="20329"/>
-<part name="U$79" library="microbuilder" deviceset="GND" device=""/>
 <part name="U$80" library="microbuilder" deviceset="GND" device=""/>
 <part name="C16" library="microbuilder" deviceset="CAP_CERAMIC" device="0805-NOOUTLINE" value="10uF"/>
@@
 <part name="GND9" library="SparkFun-PowerSymbols" library_urn="urn:adsk.eagle:library:530" deviceset="GND" device=""/>
 <part name="J2" library="SparkFun-Connectors" library_urn="urn:adsk.eagle:library:513" deviceset="CONN_07" device="NO_SILK" package3d_urn="urn:adsk.eagle:package:38136/1"/>
-<part name="H3" library="SparkFun-Hardware" library_urn="urn:adsk.eagle:library:519" deviceset="STAND-OFF" device="" package3d_urn="urn:adsk.eagle:package:38630/1"/>
-<part name="H4" library="SparkFun-Hardware" library_urn="urn:adsk.eagle:library:519" deviceset="STAND-OFF" device="" package3d_urn="urn:adsk.eagle:package:38630/1"/>
+<part name="GND15" library="SparkFun" deviceset="GND" device=""/>
+<part name="X1" library="SparkFun" deviceset="USB" device="SMD" value="Micro USB"/>
 </parts>
 <sheets>
@@
 <text x="287.02" y="-66.04" size="1.778" layer="94">RTC</text>
 <text x="193.04" y="-43.18" size="1.778" layer="94">MOTOR CONTROLER</text>
+<text x="292.354" y="90.932" size="1.778" layer="97">miniUSB</text>
 </plain>
 <instances>
@@
 <instance part="FRAME5" gate="G$2" x="467.36" y="-127"/>
 <instance part="IC4" gate="G$1" x="363.22" y="106.68"/>
-<instance part="X8" gate="G$1" x="320.04" y="96.52"/>
-<instance part="U$79" gate="G$1" x="332.74" y="86.36"/>
 <instance part="U$80" gate="G$1" x="347.98" y="106.68"/>
 <instance part="C16" gate="G$1" x="342.9" y="114.3"/>
@@
 <instance part="GND9" gate="1" x="347.98" y="35.56"/>
 <instance part="J2" gate="G$1" x="312.42" y="2.54"/>
-<instance part="H3" gate="G$1" x="398.78" y="35.56"/>
-<instance part="H4" gate="G$1" x="403.86" y="35.56"/>
+<instance part="GND15" gate="1" x="304.8" y="73.66"/>
+<instance part="X1" gate="G$1" x="299.72" y="78.74" rot="MR0"/>
 </instances>
 <busses>
@@
 <pinref part="R28" gate="G$1" pin="1"/>
 <wire x1="48.26" y1="96.52" x2="48.26" y2="99.06" width="0.1524" layer="91"/>
-</segment>
-<segment>
-<pinref part="X8" gate="G$1" pin="GND"/>
-<pinref part="U$79" gate="G$1" pin="GND"/>
-<wire x1="330.2" y1="91.44" x2="332.74" y2="91.44" width="0.1524" layer="91"/>
-<wire x1="332.74" y1="91.44" x2="332.74" y2="88.9" width="0.1524" layer="91"/>
 </segment>
 <segment>
@@
 <wire x1="416.56" y1="-20.32" x2="416.56" y2="-30.48" width="0.1524" layer="91"/>
 <pinref part="U$5" gate="G$1" pin="GND"/>
-<pinref part="J5" gate="G$1" pin="5"/>
-<wire x1="383.54" y1="-20.32" x2="416.56" y2="-20.32" width="0.1524" layer="91"/>
+<pinref part="J5" gate="G$1" pin="3"/>
+<wire x1="383.54" y1="-25.4" x2="416.56" y2="-20.32" width="0.1524" layer="91"/>
 </segment>
 <segment>
@@
 <pinref part="GND5" gate="1" pin="GND"/>
 <pinref part="C4" gate="G$1" pin="2"/>
+</segment>
+<segment>
+<wire x1="302.26" y1="78.74" x2="304.8" y2="78.74" width="0.1524" layer="91"/>
+<wire x1="304.8" y1="78.74" x2="304.8" y2="76.2" width="0.1524" layer="91"/>
+<pinref part="GND15" gate="1" pin="GND"/>
+<pinref part="X1" gate="G$1" pin="GND"/>
 </segment>
 </net>
@@
 </segment>
 <segment>
-<wire x1="403.86" y1="-30.48" x2="383.54" y2="-30.48" width="0.1524" layer="91"/>
+<wire x1="403.86" y1="-30.48" x2="383.54" y2="-17.78" width="0.1524" layer="91"/>
 <label x="388.62" y="-30.48" size="1.778" layer="95"/>
-<pinref part="J5" gate="G$1" pin="1"/>
+<pinref part="J5" gate="G$1" pin="6"/>
 </segment>
 </net>
@@
 <wire x1="393.7" y1="-17.78" x2="393.7" y2="0" width="0.1524" layer="91"/>
 <pinref part="U$4" gate="G$1" pin="3.3V"/>
-<pinref part="J5" gate="G$1" pin="6"/>
-<wire x1="383.54" y1="-17.78" x2="393.7" y2="-17.78" width="0.1524" layer="91"/>
+<pinref part="J5" gate="G$1" pin="4"/>
+<wire x1="383.54" y1="-22.86" x2="393.7" y2="-17.78" width="0.1524" layer="91"/>
 </segment>
 </net>
@@
 </segment>
 <segment>
-<wire x1="403.86" y1="-25.4" x2="383.54" y2="-25.4" width="0.1524" layer="91"/>
+<wire x1="403.86" y1="-25.4" x2="383.54" y2="-30.48" width="0.1524" layer="91"/>
 <label x="388.62" y="-25.4" size="1.778" layer="95"/>
-<pinref part="J5" gate="G$1" pin="3"/>
+<pinref part="J5" gate="G$1" pin="1"/>
 </segment>
 </net>
@@
 </segment>
 <segment>
-<pinref part="X8" gate="G$1" pin="VBUS"/>
 <pinref part="IC4" gate="G$1" pin="VBUS"/>
-<wire x1="330.2" y1="101.6" x2="335.28" y2="101.6" width="0.1524" layer="91"/>
 <wire x1="335.28" y1="101.6" x2="347.98" y2="101.6" width="0.1524" layer="91"/>
 <pinref part="U$82" gate="G$1" pin="VBUS"/>
 <wire x1="335.28" y1="101.6" x2="335.28" y2="104.14" width="0.1524" layer="91"/>
 <junction x="335.28" y="101.6"/>
+<wire x1="335.28" y1="101.6" x2="325.12" y2="101.6" width="0.1524" layer="91"/>
+<pinref part="X1" gate="G$1" pin="VBUS"/>
+<wire x1="325.12" y1="101.6" x2="325.12" y2="81.28" width="0.1524" layer="91"/>
+<wire x1="325.12" y1="81.28" x2="302.26" y2="81.28" width="0.1524" layer="91"/>
 </segment>
 <segment>
@@
 </segment>
 <segment>
-<wire x1="403.86" y1="-22.86" x2="383.54" y2="-22.86" width="0.1524" layer="91"/>
+<wire x1="403.86" y1="-22.86" x2="383.54" y2="-20.32" width="0.1524" layer="91"/>
 <label x="388.62" y="-22.86" size="1.778" layer="95"/>
-<pinref part="J5" gate="G$1" pin="4"/>
+<pinref part="J5" gate="G$1" pin="5"/>
 </segment>
 </net>
@@
 <net name="N$21" class="0">
 <segment>
-<pinref part="X8" gate="G$1" pin="D+"/>
 <pinref part="IC4" gate="G$1" pin="D+"/>
-<wire x1="330.2" y1="99.06" x2="347.98" y2="99.06" width="0.1524" layer="91"/>
+<wire x1="347.98" y1="99.06" x2="302.26" y2="99.06" width="0.1524" layer="91"/>
+<pinref part="X1" gate="G$1" pin="D+"/>
+<wire x1="302.26" y1="99.06" x2="302.26" y2="86.36" width="0.1524" layer="91"/>
 </segment>
 </net>
 <net name="N$22" class="0">
 <segment>
-<pinref part="X8" gate="G$1" pin="D-"/>
 <pinref part="IC4" gate="G$1" pin="D-"/>
-<wire x1="330.2" y1="96.52" x2="347.98" y2="96.52" width="0.1524" layer="91"/>
-</segment>
-</net>
+<wire x1="347.98" y1="96.52" x2="312.42" y2="96.52" width="0.1524" layer="91"/>
+<wire x1="312.42" y1="96.52" x2="312.42" y2="83.82" width="0.1524" layer="91"/>
+<pinref part="X1" gate="G$1" pin="D-"/>
+<wire x1="312.42" y1="83.82" x2="302.26" y2="83.82" width="0.1524" layer="91"/>
+</segment>
+</net>
