File: overallPCB.brd (EAGLE design)
At the start: 160 x 100 mm, 40 parts, among them IC1 DS3231/SO, IC4 CP2104, Q7 mmbt2222, Q8 mmbt2222, Q9 DMG3415U, SW3 KMR2, U2 TB6612 SSOP, U5 MCP73831T-2ACI/OT, U6 AP2112-3.3, X7 ESP32_WROOM32_SKINNY, X8 20329, X9 JSTPH

Commit message: Add files via upload
Parts:
- moved C16 57.7 mm to (71.1, 17.8), turned to 270 degrees
- moved R28 51.2 mm to (69.8, 33.0)
- moved Q9 48.8 mm to (71.1, 40.6), turned to 180 degrees
- moved X8 48.5 mm to (74.9, 12.7)
- moved C25 48.3 mm to (39.4, 22.9), turned to 270 degrees
- moved R23 44.2 mm to (59.7, 47.0), turned to 180 degrees
- moved Q8 44.2 mm to (76.2, 27.9)
- moved C2 42.6 mm to (43.2, 43.2), turned to 90 degrees
- moved C24 40.6 mm to (43.2, 24.1), turned to 90 degrees
- moved C21 39.2 mm to (63.5, 40.6), turned to 90 degrees
- moved R3 39.2 mm to (38.1, 43.2), turned to 270 degrees
- moved Q7 39.2 mm to (71.1, 27.9)
- moved C17 38.8 mm to (77.5, 41.9), turned to 180 degrees
- moved C20 38.6 mm to (52.1, 41.9)
- moved C22 38.2 mm to (52.1, 39.4)
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Connections:
- net 3.3V: now also J3.3; no longer J3.1
- net A0_DAC2: now also J3.1; no longer J3.6
- net CONTROL_BUTTON: now also J1.7; no longer J1.2
- net EN: now also J3.9; no longer J3.10
- net FINGERPRINT_RX: now also J1.5; no longer J1.7
- net FINGERPRINT_TX: now also J1.6; no longer J1.8
- net GND: now also J3.4; no longer J3.2
- net GPIO19: now also J3.10; no longer J3.3
- net IO13_A12: now also J3.8; no longer J3.4
- net MOTOR_C1: now also J1.1; no longer J1.9
- net MOTOR_C2: now also J1.4; no longer J1.10
- net OLED_CS: now also J1.9; no longer J1.6
- net OLED_DC: now also J1.3; no longer J1.5
- net OLED_MOSI: now also J1.10; no longer J1.4
- net OLED_SCK: now also J1.8; no longer J1.3
- net RESET: now also J3.2; no longer J3.9
- net SCANNER_BUTTON: now also J1.2; no longer J1.1
- net VBUS: now also J3.6; no longer J3.8
Routing:
- net GND: track 0.00 -> 309.2 mm, vias 0 -> 26
- net 3.3V: track 20.3 -> 159.0 mm, vias 0 -> 10
- net RESET: track 0.00 -> 92.3 mm, vias 0 -> 6
- net VBUS: track 0.00 -> 81.5 mm, vias 0 -> 7
- net IO13_A12: track 0.00 -> 58.3 mm, vias 0 -> 7
- net VBAT: track 0.00 -> 57.0 mm, vias 0 -> 8
- net A13_I35: track 0.00 -> 52.3 mm, vias 0 -> 6
- net GPIO19: track 0.00 -> 51.9 mm, vias 0 -> 7
- net A4_IO36: track 0.00 -> 44.2 mm, vias 0 -> 6
- net A0_DAC2: track 0.00 -> 41.4 mm, vias 0 -> 3
- net AIN2: track 0.00 -> 36.6 mm, vias 0 -> 2
- net VM+: track 0.00 -> 34.0 mm
- net SCL: track 4.60 -> 34.6 mm, vias 0 -> 2
- net SDA: track 7.78 -> 36.7 mm, vias 0 -> 2
- net GPIO0: track 0.00 -> 22.9 mm, vias 0 -> 4
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Other:
- board size 160 x 100 mm -> 48.2 x 47.9 mm

Commit message: Add files via upload
Parts:
- removed J2: (no value), SparkFun-Connectors:1X03_PP_HOLES_ONLY
- removed X8: 20329, microbuilder:4UCONN_20329_V2
- added H1, H2: STAND-OFF, SparkFun-Hardware:STAND-OFF
- added J4: (no value), SparkFun-Connectors:1X03
- added J5: (no value), SparkFun-Connectors:USB-B-MICRO-SMD
- moved C1 1.27 mm to (39.4, 10.2)
- moved C19 1.27 mm to (67.3, 47.0)
- moved R2 1.27 mm to (41.9, 10.2)
- moved CHG2 1.27 mm to (55.9, 45.7)
- moved J1 1.27 mm to (44.5, 8.89)
Connections:
- removed net N$21: IC4.3, X8.D+
- removed net N$22: IC4.4, X8.D-
- new net N$1: IC4.3, J5.D+
- new net N$2: IC4.4, J5.D-
- net EN: now also J3.8; no longer J3.9
- net GND: now also J5.GND; no longer X8.BASE@1, X8.BASE@2, X8.GND, X8.SPRT@1, X8.SPRT@2, X8.SPRT@3, X8.SPRT@4
- net IO13_A12: now also J3.7; no longer J3.8
- net MA1: now also J4.2; no longer J2.2
- net MA2: now also J4.3; no longer J2.1
- net VBAT: now also J3.9; no longer J3.7
- net VBUS: now also J5.VBUS; no longer X8.VBUS
- net VM+: now also J4.1; no longer J2.3
Routing:
- net GND: track 309.2 -> 281.5 mm, vias 26 -> 19
- net N$21: track 16.2 -> 0.00 mm, vias 2 -> 0
- net GPIO0: track 22.9 -> 33.3 mm
- net N$2: track 0.00 -> 8.94 mm, vias 0 -> 2
- net OLED_SCK: track 12.8 -> 21.3 mm
- net 3.3V: track 159.0 -> 166.6 mm, vias 10 -> 7
- net N$22: track 6.61 -> 0.00 mm
- net N$1: track 0.00 -> 5.86 mm
- net RESET: track 92.3 -> 97.4 mm, vias 6 -> 8
- net IO13_A12: track 58.3 -> 53.3 mm, vias 7 -> 4
- net VBUS: track 81.5 -> 86.3 mm, vias 7 -> 6
- net A13_I35: track 52.3 -> 48.0 mm, vias 6 -> 3
- net VBAT: track 57.0 -> 53.0 mm, vias 8 -> 5
- net RTS: track 12.5 -> 16.0 mm, vias 3 -> 2
- net A0_DAC2: track 41.4 -> 38.1 mm
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- added copper zone on layer 1, net GND
- added copper zone on layer 16, net GND
Other:
- board size 48.2 x 47.9 mm -> 47 x 47.9 mm
- board text added: "3.3v"
- board text added: "C1"
- board text added: "C2"
- board text added: "CBUT"
- board text added: "CS"
- board text added: "D13"
- board text added: "D19"
- board text added: "D25"
- board text added: "D26"
- board text added: "DC"
- board text added: "EN"
- board text added: "FRX"
- board text added: "FTX"
- board text added: "GND"
- board text added: "MO"
- board text added: "PICARD"
- board text added: "RES"
- board text added: "SBUT"
- board text added: "SCK"
- board text added: "VBAT"
- board text added: "VBUS"
