File: overallPCB.brd (EAGLE design)
At the start: 41.9 x 67 mm, 45 parts, among them IC1 DS3231/SO, IC4 CP2104, Q7 mmbt2222, Q8 mmbt2222, Q9 DMG3415U, SW3 KMR2, U2 TB6612 SSOP, U5 MCP73831T-2ACI/OT, U6 AP2112-3.3, X7 ESP32_WROOM32_SKINNY, X8 20329, X9 JSTPH

Commit message: Add files via upload
Parts:
- removed H3, H4: STAND-OFF, SparkFun-Hardware:STAND-OFF
- removed X8: 20329, microbuilder:4UCONN_20329_V2
- added X1: Micro USB, SparkFun:USB-MINIB
- moved C16 21.4 mm to (65.4, 38.3)
- moved R26 10.6 mm to (79.1, 50.2)
- moved C18 6.71 mm to (70.2, 50.0), turned to 270 degrees
- moved SW3 4.26 mm to (74.0, 50.1), turned to 180 degrees
- moved CHG2 3.61 mm to (88.4, 51.3)
- moved R28 3.16 mm to (79.7, 44.0)
- moved C17 2.69 mm to (86.6, 48.3)
- moved J5 2.50 mm to (74.2, 56.1)
- moved R23 1.12 mm to (81.8, 46.0)
- moved R22 1.00 mm to (83.8, 46.0)
- moved H1 0.71 mm to (98.6, 55.1)
- moved H2 0.71 mm to (64.3, 55.1)
- moved R27 0.50 mm to (78.7, 40.1)
Connections:
- net 3.3V: now also J5.4; no longer J5.6
- net EN: now also J5.5; no longer J5.4
- net GND: now also J5.3, X1.GND; no longer J5.5, X8.BASE@1, X8.BASE@2, X8.GND, X8.SPRT@1, X8.SPRT@2, X8.SPRT@3, X8.SPRT@4
- net N$21: now also X1.D+; no longer X8.D+
- net N$22: now also X1.D-; no longer X8.D-
- net RESET: now also J5.1; no longer J5.3
- net VBAT: now also J5.6; no longer J5.1
- net VBUS: now also X1.VBUS; no longer X8.VBUS
Routing:
- net GND: track 189.3 -> 307.2 mm, vias 11 -> 17
- net VBUS: track 17.6 -> 63.9 mm, vias 2 -> 6
- net RESET: track 62.6 -> 107.0 mm, vias 3 -> 4
- net 3.3V: track 156.9 -> 186.1 mm, vias 8 -> 7
- net EN: track 2.55 -> 20.7 mm, vias 0 -> 1
- net VBAT: track 21.9 -> 36.7 mm
- net N$21: track 0.00 -> 12.9 mm
- net N$22: track 0.00 -> 12.1 mm, vias 0 -> 2
- net A13_I35: track 39.5 -> 37.4 mm
- net VM+: track 35.9 -> 34.2 mm
- net N$26: track 14.5 -> 13.1 mm
- net N$23: track 1.91 -> 3.00 mm
- added copper zone on layer 1, net GND
- added copper zone on layer 16, net GND
Other:
- board size 41.9 x 67 mm -> 41.9 x 58.5 mm
- board text added: "3.3"
- board text added: "PICARD"
- board text added: "a0"
- board text added: "c1"
- board text added: "c2"
- board text added: "cBtn"
- board text added: "cs"
- board text added: "dc"
- board text added: "en"
- board text added: "fngTx"
- board text added: "gnd"
- board text added: "io13"
- board text added: "io19"
- board text added: "ma1"
- board text added: "ma2"
- board text added: "mo"
- board text added: "res"
- board text added: "sBtn"
- board text added: "sck"
- board text added: "tx"
- board text added: "vbat"
- board text added: "vbus"
- board text added: "vm"

Commit message: Add files via upload
Other:
- board size 41.9 x 58.5 mm -> 42 x 58.5 mm
Changed lines of the file:
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@@
 <board>
 <plain>
-<wire x1="60.96" y1="58.36" x2="60.96" y2="-0.12" width="0" layer="20"/>
-<wire x1="60.96" y1="-0.12" x2="70.88" y2="-0.12" width="0" layer="20"/>
-<wire x1="70.88" y1="-0.12" x2="77" y2="0" width="0" layer="20"/>
-<wire x1="77" y1="0" x2="77" y2="6" width="0" layer="20"/>
+<wire x1="61" y1="58.36" x2="61" y2="0.5" width="0" layer="20"/>
+<wire x1="61" y1="0.5" x2="77" y2="0.5" width="0" layer="20"/>
+<wire x1="77" y1="0.5" x2="77" y2="6" width="0" layer="20"/>
 <wire x1="77" y1="6" x2="96" y2="6" width="0" layer="20"/>
 <wire x1="96" y1="6" x2="96" y2="0" width="0" layer="20"/>
-<wire x1="96" y1="0" x2="96.5" y2="0" width="0" layer="20"/>
-<wire x1="96.5" y1="0" x2="102.85" y2="-0.12" width="0" layer="20"/>
-<wire x1="102.85" y1="-0.12" x2="102.85" y2="58.36" width="0" layer="20"/>
-<wire x1="102.85" y1="58.36" x2="60.96" y2="58.36" width="0" layer="20"/>
+<wire x1="96" y1="0" x2="103" y2="0" width="0" layer="20"/>
+<wire x1="103" y1="0" x2="103" y2="58.5" width="0" layer="20"/>
+<wire x1="103" y1="58.5" x2="61" y2="58.5" width="0" layer="20"/>
+<wire x1="61" y1="58.5" x2="61" y2="58.36" width="0" layer="20"/>
+<wire x1="61" y1="58.36" x2="60.96" y2="58.36" width="0" layer="20"/>
 <dimension x1="61" y1="59.5" x2="103" y2="59.5" x3="82" y3="61" textsize="1.778" layer="51" dtype="horizontal" unit="inch" precision="6"/>
 <dimension x1="57.5" y1="0" x2="57.5" y2="58.5" x3="57.5" y3="29.25" textsize="1.778" layer="51" dtype="horizontal" unit="inch" precision="6"/>
@@
 <wire x1="77.086" y1="33.586" x2="77.086" y2="36.167875" width="0.254" layer="1"/>
 <wire x1="76.2" y1="32.7" x2="77.086" y2="33.586" width="0.254" layer="1"/>
-<polygon width="0.254" layer="1" isolate="0.3048">
+<polygon width="0.1524" layer="16" isolate="0.3048">
+<vertex x="96" y="6"/>
+<vertex x="77" y="6"/>
+<vertex x="77" y="0.5"/>
+<vertex x="61" y="0.5"/>
+<vertex x="61" y="1"/>
 <vertex x="61" y="58.5"/>
 <vertex x="103" y="58.5"/>
+<vertex x="103" y="57.5"/>
 <vertex x="103" y="0"/>
-<vertex x="96.5" y="0"/>
+<vertex x="102.5" y="0"/>
 <vertex x="96" y="0"/>
+</polygon>
+<polygon width="0.1524" layer="1" isolate="0.3048">
+<vertex x="77" y="6"/>
 <vertex x="96" y="6"/>
-<vertex x="77" y="6"/>
-<vertex x="77" y="0"/>
-<vertex x="61" y="0"/>
-</polygon>
-<polygon width="0.254" layer="16" isolate="0.3048">
+<vertex x="96" y="0"/>
+<vertex x="103" y="0"/>
+<vertex x="103" y="58.5"/>
 <vertex x="61" y="58.5"/>
-<vertex x="103" y="58.5"/>
-<vertex x="103" y="0"/>
-<vertex x="96" y="0"/>
-<vertex x="96" y="6"/>
-<vertex x="77" y="6"/>
-<vertex x="77" y="0"/>
-<vertex x="61" y="0"/>
+<vertex x="61" y="57"/>
+<vertex x="61" y="0.5"/>
+<vertex x="77" y="0.5"/>
 </polygon>
 </signal>
